File: Board/KiCAD/Battery_Management_System.kicad_pcb (KiCad board)
At the start: 2 copper layers, 0 parts

Commit message: Added project libraries that were previously committed
Other:
- board outline added: 40 x 50 mm
- copper layers 2 -> 4
Changed lines of the file:
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@@
 	(generator_version "9.0")
 	(general
-		(thickness 1.6)
+		(thickness 1.7702)
 		(legacy_teardrops no)
 	)
@@
 	(layers
 		(0 "F.Cu" signal)
+		(4 "In1.Cu" signal)
+		(6 "In2.Cu" signal)
 		(2 "B.Cu" signal)
-		(9 "F.Adhes" user "F.Adhesive")
-		(11 "B.Adhes" user "B.Adhesive")
 		(13 "F.Paste" user)
 		(15 "B.Paste" user)
@@
 		(17 "Dwgs.User" user "User.Drawings")
 		(19 "Cmts.User" user "User.Comments")
-		(21 "Eco1.User" user "User.Eco1")
-		(23 "Eco2.User" user "User.Eco2")
 		(25 "Edge.Cuts" user)
 		(27 "Margin" user)
@@
 		(35 "F.Fab" user)
 		(33 "B.Fab" user)
-		(39 "User.1" user)
-		(41 "User.2" user)
-		(43 "User.3" user)
-		(45 "User.4" user)
 	)
 	(setup
+		(stackup
+			(layer "F.SilkS"
+				(type "Top Silk Screen")
+				(color "White")
+				(material "Liquid Photo")
+			)
+			(layer "F.Paste"
+				(type "Top Solder Paste")
+			)
+			(layer "F.Mask"
+				(type "Top Solder Mask")
+				(color "Purple")
+				(thickness 0.0254)
+				(material "Liquid Ink")
+				(epsilon_r 3.3)
+				(loss_tangent 0)
+			)
+			(layer "F.Cu"
+				(type "copper")
+				(thickness 0.0432)
+			)
+			(layer "dielectric 1"
+				(type "prepreg")
+				(thickness 0.2021)
+				(material "FR408-HR")
+				(epsilon_r 3.69)
+				(loss_tangent 0.0091)
+			)
+			(layer "In1.Cu"
+				(type "copper")
+				(thickness 0.0175)
+			)
+			(layer "dielectric 2"
+				(type "core")
+				(thickness 1.1938)
+				(material "FR408-HR")
+				(epsilon_r 3.69)
+				(loss_tangent 0.0091)
+			)
+			(layer "In2.Cu"
+				(type "copper")
+				(thickness 0.0175)
+			)
+			(layer "dielectric 3"
+				(type "prepreg")
+				(thickness 0.2021)
+				(material "FR408-HR")
+				(epsilon_r 3.69)
+				(loss_tangent 0.0091)
+			)
+			(layer "B.Cu"
+				(type "copper")
+				(thickness 0.0432)
+			)
+			(layer "B.Mask"
+				(type "Bottom Solder Mask")
+				(color "Purple")
+				(thickness 0.0254)
+				(material "Liquid Ink")
+				(epsilon_r 3.3)
+				(loss_tangent 0)
+			)
+			(layer "B.Paste"
+				(type "Bottom Solder Paste")
+			)
+			(layer "B.SilkS"
+				(type "Bottom Silk Screen")
+				(color "White")
+				(material "Liquid Photo")
+			)
+			(copper_finish "ENIG")
+			(dielectric_constraints no)
+		)
 		(pad_to_mask_clearance 0)
 		(allow_soldermask_bridges_in_footprints no)
@@
 	)
 	(net 0 "")
+	(gr_rect
+		(start 170 130)
+		(end 210 180)
+		(stroke
+			(width 0.1)
+			(type default)
+		)
+		(fill no)
+		(layer "Edge.Cuts")
+	)
 	(embedded_fonts no)
 )

Commit message: Add files via upload
Parts:
- added C10: 10uF, Capacitor_SMD:C_0201_0603Metric, F.Cu at (118.7, 64.9)
- added C12: 10uF, Capacitor_SMD:C_0201_0603Metric, F.Cu at (118.7, 66.7)
- added C13: 1uF, Capacitor_SMD:C_0201_0603Metric, F.Cu at (118.7, 68.4)
- added C14: 47nF, Capacitor_SMD:C_0201_0603Metric, F.Cu at (118.7, 70.2)
- added C15: 47nF, Capacitor_SMD:C_0201_0603Metric, F.Cu at (118.7, 71.9)
- added C22: 10uF, Capacitor_SMD:C_0201_0603Metric, F.Cu at (118.7, 73.7)
- added C23: 0.1uF, Capacitor_SMD:C_0201_0603Metric, F.Cu at (118.7, 75.4)
- added C24: 0.1uF, Capacitor_SMD:C_0201_0603Metric, F.Cu at (121.1, 61.4)
- added C25: 10uF, Capacitor_SMD:C_0201_0603Metric, F.Cu at (121.1, 63.2)
- added C26: 3.3uF, Capacitor_SMD:C_0201_0603Metric, F.Cu at (121.1, 64.9)
- added C27: 100pF, Capacitor_SMD:C_0201_0603Metric, F.Cu at (121.1, 66.7)
- added C28: 10uF, Capacitor_SMD:C_0201_0603Metric, F.Cu at (121.1, 68.4)
- added C29: 10uF, Capacitor_SMD:C_0201_0603Metric, F.Cu at (121.1, 70.2)
- added C30: 20pF, Capacitor_SMD:C_0201_0603Metric, F.Cu at (118.7, 109.8)
- added C31: 20pF, Capacitor_SMD:C_0201_0603Metric, F.Cu at (118.7, 111.6)
- added C32: 20pF, Capacitor_SMD:C_0201_0603Metric, F.Cu at (118.7, 113.3)
- added C33: 20pF, Capacitor_SMD:C_0201_0603Metric, F.Cu at (118.7, 115.1)
- added C34: 100nF, Capacitor_SMD:C_0201_0603Metric, F.Cu at (121.1, 109.8)
- added C35: 100pF, Capacitor_SMD:C_0201_0603Metric, F.Cu at (121.1, 71.9)
- added C36: 33pF, Capacitor_SMD:C_0201_0603Metric, F.Cu at (121.1, 73.7)
- added C37: 15pF, Capacitor_SMD:C_0201_0603Metric, F.Cu at (121.1, 75.4)
- added C38: 4.7nF, Capacitor_SMD:C_0201_0603Metric, F.Cu at (123.6, 61.4)
- added C39: 680pF, Capacitor_SMD:C_0201_0603Metric, F.Cu at (123.6, 63.2)
- added C40: 1uF, Capacitor_SMD:C_0201_0603Metric, F.Cu at (123.6, 64.9)
- added C41: 10nF, Capacitor_SMD:C_0201_0603Metric, F.Cu at (123.6, 66.7)
- added C42: 33nF, Capacitor_SMD:C_0201_0603Metric, F.Cu at (123.6, 68.4)
- added C43: 33nF, Capacitor_SMD:C_0201_0603Metric, F.Cu at (123.6, 70.2)
- added C44: 33uF, Capacitor_SMD:C_0201_0603Metric, F.Cu at (123.6, 71.9)
- added C45: 33uF, Capacitor_SMD:C_0201_0603Metric, F.Cu at (123.6, 73.7)
- added C47: 100n, Capacitor_SMD:C_0201_0603Metric, F.Cu at (109.3, 90.7)
- added C48: 100n, Capacitor_SMD:C_0201_0603Metric, F.Cu at (109.3, 92.4)
- added C49: 100n, Capacitor_SMD:C_0201_0603Metric, F.Cu at (109.3, 94.2)
- added C50: 100n, Capacitor_SMD:C_0201_0603Metric, F.Cu at (109.3, 95.9)
- added C51: 2.2uF, Capacitor_SMD:C_0201_0603Metric, F.Cu at (121.1, 111.6)
- added C52: 10uF, Capacitor_SMD:C_0201_0603Metric, F.Cu at (121.1, 113.3)
- added C53: 10uF, Capacitor_SMD:C_0201_0603Metric, F.Cu at (121.1, 115.1)
- added C7: 1nF, Capacitor_SMD:C_0201_0603Metric, F.Cu at (118.7, 61.4)
- added C9: 10nF, Capacitor_SMD:C_0201_0603Metric, F.Cu at (118.7, 63.2)
- added J1: Conn_01x06_Socket, Connector_PinHeader_1.00mm:PinHeader_1x06_P1.00mm_Vertical, F.Cu at (87.6, 135.2)
- added J2: Conn_ARM_SWD_TagConnect_TC2030, Connector:Tag-Connect_TC2030-IDC-FP_2x03_P1.27mm_Vertical, F.Cu at (135.4, 107.1)
- added J4: Conn_01x03, Connector_PinHeader_1.00mm:PinHeader_1x03_P1.00mm_Vertical, F.Cu at (126.5, 110.5)
- added J5: Conn_01x03, Connector_PinHeader_1.00mm:PinHeader_1x03_P1.00mm_Vertical, F.Cu at (94.3, 139.2)
- added J7: Conn_01x05, Connector_PinHeader_1.00mm:PinHeader_1x05_P1.00mm_Vertical, F.Cu at (91.0, 139.2)
- added J8: Conn_01x02, Connector_PinHeader_1.00mm:PinHeader_1x02_P1.00mm_Vertical, F.Cu at (91.0, 135.2)
- added J9: Conn_01x02, Connector_PinHeader_1.00mm:PinHeader_1x02_P1.00mm_Vertical, F.Cu at (94.3, 135.2)
- added L2: 4.7uH, Inductor_SMD:L_10.4x10.4_H4.8, F.Cu at (136.0, 66.5)
- added L3: 3.3uH, Inductor_SMD:L_10.4x10.4_H4.8, F.Cu at (123.7, 96.3)
- added Q1: AON7408, AON7408:TRANS_AON7408, F.Cu at (140.9, 74.9)
- added Q10: AON7407, AON7407:TRANS_AON7407, F.Cu at (120.4, 85.2)
- added Q2: AON6500, AON6500:TRANS_AON6500, F.Cu at (134.2, 75.9)
- added Q23: 2N7002, Package_TO_SOT_SMD:SOT-23, F.Cu at (105.7, 92.2)
- added Q24: 2N7002, Package_TO_SOT_SMD:SOT-23, F.Cu at (105.7, 96.8)
- added Q25: 2N7002, Package_TO_SOT_SMD:SOT-23, F.Cu at (105.7, 101.5)
- added Q26: 2N7002, Package_TO_SOT_SMD:SOT-23, F.Cu at (105.7, 106.1)
- added Q27: IRF9540NSTRLPBF, IRF9540NSTRLPBF:DPAK254P1524X483-4_3N, F.Cu at (52.8, 58.4)
- added Q28: IRF9540NSTRLPBF, IRF9540NSTRLPBF:DPAK254P1524X483-4_3N, F.Cu at (52.8, 70.7)
- added Q29: IRF9540NSTRLPBF, IRF9540NSTRLPBF:DPAK254P1524X483-4_3N, F.Cu at (52.8, 82.9)
- added Q3: AON7408, AON7408:TRANS_AON7408, F.Cu at (140.9, 79.6)
- added Q30: IRF9540NSTRLPBF, IRF9540NSTRLPBF:DPAK254P1524X483-4_3N, F.Cu at (52.8, 95.1)
- added Q4: AON6500, AON6500:TRANS_AON6500, F.Cu at (134.2, 82.6)
- added R10: 30k, Resistor_SMD:R_0201_0603Metric, F.Cu at (126.0, 73.7)
- added R15: 10k, Resistor_SMD:R_0201_0603Metric, F.Cu at (126.0, 75.4)
- added R17: 10k, Resistor_SMD:R_0201_0603Metric, F.Cu at (109.3, 97.7)
- added R2: 10m, Resistor_SMD:R_0201_0603Metric, F.Cu at (123.6, 75.4)
- added R3: 2.2m, Resistor_SMD:R_0201_0603Metric, F.Cu at (126.0, 61.4)
- added R35: 10k, Resistor_SMD:R_0201_0603Metric, F.Cu at (128.5, 61.4)
- added R36: 15k, Resistor_SMD:R_0201_0603Metric, F.Cu at (128.5, 63.2)
- added R37: 39k, Resistor_SMD:R_0201_0603Metric, F.Cu at (128.5, 64.9)
- added R38: 220k, Resistor_SMD:R_0201_0603Metric, F.Cu at (128.5, 66.7)
- added R39: 380k, Resistor_SMD:R_0201_0603Metric, F.Cu at (128.5, 68.4)
- added R4: 10m, Resistor_SMD:R_0201_0603Metric, F.Cu at (126.0, 63.2)
- added R40: 10, Resistor_SMD:R_0201_0603Metric, F.Cu at (128.5, 70.2)
- added R41: 5,1, Resistor_SMD:R_0201_0603Metric, F.Cu at (128.5, 71.9)
- added R42: 5.1, Resistor_SMD:R_0201_0603Metric, F.Cu at (128.5, 73.7)
- added R5: 10, Resistor_SMD:R_0201_0603Metric, F.Cu at (126.0, 64.9)
- added R58: 100k, Resistor_SMD:R_0201_0603Metric, F.Cu at (123.6, 109.8)
- added R6: 10, Resistor_SMD:R_0201_0603Metric, F.Cu at (126.0, 66.7)
- added R60: 4.7k, Resistor_SMD:R_0201_0603Metric, F.Cu at (123.6, 111.6)
- added R62: 10k, Resistor_SMD:R_0201_0603Metric, F.Cu at (109.3, 99.4)
- added R63: 10k, Resistor_SMD:R_0201_0603Metric, F.Cu at (111.8, 90.7)
- added R64: 10k, Resistor_SMD:R_0201_0603Metric, F.Cu at (111.8, 92.4)
- added R65: 10k, Resistor_SMD:R_0201_0603Metric, F.Cu at (111.8, 94.2)
- added R66: 10k, Resistor_SMD:R_0201_0603Metric, F.Cu at (111.8, 95.9)
- added R67: 10k, Resistor_SMD:R_0201_0603Metric, F.Cu at (111.8, 97.7)
- added R68: 10k, Resistor_SMD:R_0201_0603Metric, F.Cu at (111.8, 99.4)
- added R69: 10k, Resistor_SMD:R_0201_0603Metric, F.Cu at (114.2, 90.7)
- added R7: 350k, Resistor_SMD:R_0201_0603Metric, F.Cu at (126.0, 68.4)
- added R70: 10k, Resistor_SMD:R_0201_0603Metric, F.Cu at (114.2, 92.4)
- added R71: 10k, Resistor_SMD:R_0201_0603Metric, F.Cu at (114.2, 94.2)
- added R72: 10k, Resistor_SMD:R_0201_0603Metric, F.Cu at (114.2, 95.9)
- added R74: R_Small, Resistor_SMD:R_0201_0603Metric, F.Cu at (114.2, 97.7)
- added R75: 4.7k, Resistor_SMD:R_0201_0603Metric, F.Cu at (123.6, 113.3)
- added R76: 50m, Resistor_SMD:R_1206_3216Metric, F.Cu at (125.6, 84.5)
- added R8: 350k, Resistor_SMD:R_0201_0603Metric, F.Cu at (126.0, 70.2)
- added R9: 200k, Resistor_SMD:R_0201_0603Metric, F.Cu at (126.0, 71.9)
- added SW2: SW_Push, Button_Switch_SMD:SW_Push_1P1T_NO_CK_KMR2, F.Cu at (133.9, 114.2)
- added U1: BQ25730RSNR, BQ25730RSNR:IC_BQ25730RSNR, F.Cu at (141.7, 85.2)
- added U3: LTC2943CDD_PBF, Package_SO:SOIC-8-1EP_3.9x4.9mm_P1.27mm_EP2.29x3mm, F.Cu at (121.7, 79.6)
- added U4: INA260, Package_SO:TSSOP-16_4.4x5mm_P0.65mm, F.Cu at (108.0, 66.7)
- added U5: LMR50410, Package_TO_SOT_SMD:SOT-23-6, F.Cu at (139.8, 114.3)
- added U6: INA260, Package_SO:TSSOP-16_4.4x5mm_P0.65mm, F.Cu at (108.0, 73.3)
- added U7: INA260, Package_SO:TSSOP-16_4.4x5mm_P0.65mm, F.Cu at (108.0, 79.9)
- added U8: INA260, Package_SO:TSSOP-16_4.4x5mm_P0.65mm, F.Cu at (108.0, 86.5)
- added U9: STM32F103C8T6, STM32F103C8T6:QFP50P900X900X160-48N, F.Cu at (136.8, 96.1)
- added Y4: CM8V-T1A-32.768KHZ-12.5PF-20PPM-TA-QA, CM8V-T1A-32.768KHZ:XTAL_CM8V-T1A-32.768KHZ-12.5PF-20PPM-TA-QA, F.Cu at (141.6, 103.8)
- added Y5: 8MHz, Crystal:Crystal_HC49-4H_Vertical, F.Cu at (121.6, 105.6)
Other:
- board outline removed

Commit message: Add files via upload
Parts:
- removed Q27, Q28, Q29, Q30: IRF9540NSTRLPBF, IRF9540NSTRLPBF:DPAK254P1524X483-4_3N
- added Q5: BSS83P, Package_TO_SOT_SMD:SOT-23, F.Cu at (237.5, 142.9)
- added Q6: BSS83P, Package_TO_SOT_SMD:SOT-23, F.Cu at (237.5, 149.0)
- added Q7: BSS83P, Package_TO_SOT_SMD:SOT-23, F.Cu at (237.6, 155.1)
- added Q8: BSS83P, Package_TO_SOT_SMD:SOT-23, F.Cu at (237.8, 161.5)
- L3: footprint Inductor_SMD:L_10.4x10.4_H4.8 -> Inductor_SMD:L_1008_2520Metric_Pad1.43x2.20mm_HandSolder
- moved J7 152.2 mm to (241.9, 158.3)
- moved J8 149.9 mm to (240.9, 134.9)
- moved J5 147.2 mm to (240.7, 123.2)
- moved J9 146.7 mm to (240.9, 129.8)
- moved Q23 144.8 mm to (232.8, 161.5)
- moved R66 140.2 mm to (235.3, 162.4), turned to 90 degrees
- moved U4 140.1 mm to (225.7, 142.7)
- moved R62 140.0 mm to (235.3, 160.6), turned to 90 degrees
- moved U6 140.0 mm to (225.7, 149.0)
- moved U7 139.9 mm to (225.7, 155.4)
- moved U8 139.8 mm to (225.9, 161.7)
- moved Q24 139.8 mm to (232.7, 155.1)
- moved C47 139.7 mm to (230.3, 160.6), turned to 90 degrees
- moved R17 137.2 mm to (230.3, 162.3), turned to 90 degrees
- moved R70 136.6 mm to (235.2, 156.0), turned to 90 degrees
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Routing:
- added copper zone on B.Cu, net (none)
- added copper zone on F.Cu, net (none)
- added copper zone on In1.Cu, net (none)
- added copper zone on In2.Cu, net (none)
Other:
- board text added: "Cell Balancer cluster"
- board text added: "Charge cluster"
- board text added: "Microcontroller CLuster"

Commit message: Add files via upload
Parts:
- removed C7: 1nF, Capacitor_SMD:C_0201_0603Metric
- C10, C12, C22, C25, C28, C29, C52, C53: footprint Capacitor_SMD:C_0201_0603Metric -> Capacitor_SMD:C_1206_3216Metric
- C13, C14, C15, C23, C24, C26, C27, C30, C31, C32, C33, C34, C35, C36, C37, C38, C39, C40, C41, C42, C43, C44, C45, C47, C48, C49, C50, C51, C9: footprint Capacitor_SMD:C_0201_0603Metric -> Capacitor_SMD:C_0603_1608Metric
- J1: footprint Connector_PinHeader_1.00mm:PinHeader_1x06_P1.00mm_Vertical -> Connector_PinHeader_2.54mm:PinHeader_1x06_P2.54mm_Vertical
- J4, J5: footprint Connector_PinHeader_1.00mm:PinHeader_1x03_P1.00mm_Vertical -> Connector_PinHeader_2.54mm:PinHeader_1x03_P2.54mm_Vertical
- J7: footprint Connector_PinHeader_1.00mm:PinHeader_1x05_P1.00mm_Vertical -> Connector_PinHeader_2.54mm:PinHeader_1x05_P2.54mm_Vertical
- J8, J9: footprint Connector_PinHeader_1.00mm:PinHeader_1x02_P1.00mm_Vertical -> Connector_PinHeader_2.54mm:PinHeader_1x02_P2.54mm_Vertical
- Q2, Q4: value AON6500 -> AON7408; footprint AON6500:TRANS_AON6500 -> AON7408:TRANS_AON7408
- R10, R15, R17, R35, R36, R37, R38, R39, R40, R41, R42, R5, R58, R6, R60, R62, R63, R64, R65, R66, R67, R68, R69, R7, R70, R71, R72, R74, R75, R8, R9: footprint Resistor_SMD:R_0201_0603Metric -> Resistor_SMD:R_0603_1608Metric
- R2, R4: footprint Resistor_SMD:R_0201_0603Metric -> Resistor_SMD:R_1206_3216Metric
- R3: value 2.2m -> 2.2; footprint Resistor_SMD:R_0201_0603Metric -> Resistor_SMD:R_0603_1608Metric
- moved C10 98.6 mm to (212.6, 55.1), turned to -90 degrees
- moved C12 97.7 mm to (215.1, 55.1), turned to -90 degrees
- moved R2 96.5 mm to (217.5, 55.1), turned to -90 degrees
- moved R15 89.8 mm to (221.9, 66.0), turned to 180 degrees
- moved R35 88.4 mm to (221.9, 64.3), turned to 180 degrees
- moved C9 88.0 mm to (210.7, 61.0), turned to -90 degrees
- moved C35 87.5 mm to (221.9, 67.6), turned to 180 degrees
- moved R9 86.7 mm to (221.9, 69.3), turned to 180 degrees
- moved U1 86.2 mm to (226.6, 66.7), turned to 0 degrees
- moved Q2 85.3 mm to (218.1, 60.3), turned to 90 degrees
- moved J4 84.9 mm to (325.5, 119.7)
- moved Q1 84.6 mm to (214.2, 60.3), turned to 90 degrees
- moved C27 83.5 mm to (224.5, 71.0), turned to -90 degrees
- moved R10 82.9 mm to (226.2, 71.0), turned to -90 degrees
- moved J9 82.1 mm to (209.6, 53.9)
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Other:
- board text removed: "Charge cluster"

Commit message: Update Battery_Management_System.kicad_pcb
Parts:
- moved C36 45.1 mm to (229.6, 99.4)
- moved C37 45.1 mm to (231.4, 101.8)
- moved C38 45.1 mm to (229.6, 97.8)
- moved C39 45.1 mm to (231.4, 103.4)
- moved C40 45.1 mm to (222.1, 112.3)
- moved C41 45.1 mm to (218.0, 107.0)
- moved C42 45.1 mm to (217.4, 109.5)
- moved C43 45.1 mm to (217.3, 108.6)
- moved C44 45.1 mm to (212.5, 101.1)
- moved C45 45.1 mm to (212.5, 102.1)
- moved R3 45.1 mm to (215.8, 110.5)
- moved R37 45.1 mm to (232.0, 98.6)
- moved R38 45.1 mm to (220.8, 111.8)
- moved R41 45.1 mm to (216.7, 107.4)
- moved R42 45.1 mm to (216.7, 106.6)
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Changed lines of the file:
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@@
 	(footprint "Resistor_SMD:R_0603_1608Metric"
 		(layer "F.Cu")
-		(at 192.3796 120.3076 -90)
+		(at 233.8448 102.6292 -90)
 		(descr "Resistor SMD 0603 (1608 Metric), square (rectangular) end terminal, IPC-7351 nominal, (Body size source: IPC-SM-782 page 72, https://www.pcb-3d.com/wordpress/wp-content/uploads/ipc-sm-782a_amendment_1_and_2.pdf), generated with kicad-footprint-generator")
 		(tags "resistor")
@@
 	(footprint "Capacitor_SMD:C_0603_1608Metric"
 		(layer "F.Cu")
-		(at 171.033 119.7864)
+		(at 212.4982 102.108)
 		(descr "Capacitor SMD 0603 (1608 Metric), square (rectangular) end terminal, IPC-7351 nominal, (Body size source: IPC-SM-782 page 76, https://www.pcb-3d.com/wordpress/wp-content/uploads/ipc-sm-782a_amendment_1_and_2.pdf), generated with kicad-footprint-generator")
 		(tags "capacitor")
@@
 	(footprint "Resistor_SMD:R_0603_1608Metric"
 		(layer "F.Cu")
-		(at 175.2648 124.2728)
+		(at 216.73 106.5944)
 		(descr "Resistor SMD 0603 (1608 Metric), square (rectangular) end terminal, IPC-7351 nominal, (Body size source: IPC-SM-782 page 72, https://www.pcb-3d.com/wordpress/wp-content/uploads/ipc-sm-782a_amendment_1_and_2.pdf), generated with kicad-footprint-generator")
 		(tags "resistor")
@@
 	(footprint "Resistor_SMD:R_0603_1608Metric"
 		(layer "F.Cu")
-		(at 182.067 129.4572 90)
+		(at 223.5322 111.7788 90)
 		(descr "Resistor SMD 0603 (1608 Metric), square (rectangular) end terminal, IPC-7351 nominal, (Body size source: IPC-SM-782 page 72, https://www.pcb-3d.com/wordpress/wp-content/uploads/ipc-sm-782a_amendment_1_and_2.pdf), generated with kicad-footprint-generator")
 		(tags "resistor")
@@
 	(footprint "Resistor_SMD:R_0603_1608Metric"
 		(layer "F.Cu")
-		(at 175.2542 125.0856)
+		(at 216.7194 107.4072)
 		(descr "Resistor SMD 0603 (1608 Metric), square (rectangular) end terminal, IPC-7351 nominal, (Body size source: IPC-SM-782 page 72, https://www.pcb-3d.com/wordpress/wp-content/uploads/ipc-sm-782a_amendment_1_and_2.pdf), generated with kicad-footprint-generator")
 		(tags "resistor")
@@
 	(footprint "Capacitor_SMD:C_0603_1608Metric"
 		(layer "F.Cu")
-		(at 188.1756 115.4694 180)
+		(at 229.6408 97.791 180)
 		(descr "Capacitor SMD 0603 (1608 Metric), square (rectangular) end terminal, IPC-7351 nominal, (Body size source: IPC-SM-782 page 76, https://www.pcb-3d.com/wordpress/wp-content/uploads/ipc-sm-782a_amendment_1_and_2.pdf), generated with kicad-footprint-generator")
 		(tags "capacitor")
@@
 	(footprint "Capacitor_SMD:C_0603_1608Metric"
 		(layer "F.Cu")
-		(at 176.5094 124.694 90)
+		(at 217.9746 107.0156 90)
 		(descr "Capacitor SMD 0603 (1608 Metric), square (rectangular) end terminal, IPC-7351 nominal, (Body size source: IPC-SM-782 page 76, https://www.pcb-3d.com/wordpress/wp-content/uploads/ipc-sm-782a_amendment_1_and_2.pdf), generated with kicad-footprint-generator")
 		(tags "capacitor")
@@
 	(footprint "Resistor_SMD:R_0603_1608Metric"
 		(layer "F.Cu")
-		(at 178.4094 129.4466 90)
+		(at 219.8746 111.7682 90)
 		(descr "Resistor SMD 0603 (1608 Metric), square (rectangular) end terminal, IPC-7351 nominal, (Body size source: IPC-SM-782 page 72, https://www.pcb-3d.com/wordpress/wp-content/uploads/ipc-sm-782a_amendment_1_and_2.pdf), generated with kicad-footprint-generator")
 		(tags "resistor")
@@
 	(footprint "Capacitor_SMD:C_0603_1608Metric"
 		(layer "F.Cu")
-		(at 175.8892 127.2192)
+		(at 217.3544 109.5408)
 		(descr "Capacitor SMD 0603 (1608 Metric), square (rectangular) end terminal, IPC-7351 nominal, (Body size source: IPC-SM-782 page 76, https://www.pcb-3d.com/wordpress/wp-content/uploads/ipc-sm-782a_amendment_1_and_2.pdf), generated with kicad-footprint-generator")
 		(tags "capacitor")
@@
 	(footprint "Capacitor_SMD:C_0603_1608Metric"
 		(layer "F.Cu")
-		(at 175.9404 128.1336)
+		(at 217.4056 110.4552)
 		(descr "Capacitor SMD 0603 (1608 Metric), square (rectangular) end terminal, IPC-7351 nominal, (Body size source: IPC-SM-782 page 76, https://www.pcb-3d.com/wordpress/wp-content/uploads/ipc-sm-782a_amendment_1_and_2.pdf), generated with kicad-footprint-generator")
 		(tags "capacitor")
@@
 	(footprint "Resistor_SMD:R_0603_1608Metric"
 		(layer "F.Cu")
-		(at 179.3588 129.4442 90)
+		(at 220.824 111.7658 90)
 		(descr "Resistor SMD 0603 (1608 Metric), square (rectangular) end terminal, IPC-7351 nominal, (Body size source: IPC-SM-782 page 72, https://www.pcb-3d.com/wordpress/wp-content/uploads/ipc-sm-782a_amendment_1_and_2.pdf), generated with kicad-footprint-generator")
 		(tags "resistor")
@@
 	(footprint "Capacitor_SMD:C_0603_1608Metric"
 		(layer "F.Cu")
-		(at 175.8688 126.2286)
+		(at 217.334 108.5502)
 		(descr "Capacitor SMD 0603 (1608 Metric), square (rectangular) end terminal, IPC-7351 nominal, (Body size source: IPC-SM-782 page 76, https://www.pcb-3d.com/wordpress/wp-content/uploads/ipc-sm-782a_amendment_1_and_2.pdf), generated with kicad-footprint-generator")
 		(tags "capacitor")
@@
 	(footprint "Capacitor_SMD:C_0603_1608Metric"
 		(layer "F.Cu")
-		(at 189.9536 121.0818 180)
+		(at 231.4188 103.4034 180)
 		(descr "Capacitor SMD 0603 (1608 Metric), square (rectangular) end terminal, IPC-7351 nominal, (Body size source: IPC-SM-782 page 76, https://www.pcb-3d.com/wordpress/wp-content/uploads/ipc-sm-782a_amendment_1_and_2.pdf), generated with kicad-footprint-generator")
 		(tags "capacitor")
@@
 	(footprint "Capacitor_SMD:C_0603_1608Metric"
 		(layer "F.Cu")
-		(at 170.9974 118.806)
+		(at 212.4626 101.1276)
 		(descr "Capacitor SMD 0603 (1608 Metric), square (rectangular) end terminal, IPC-7351 nominal, (Body size source: IPC-SM-782 page 76, https://www.pcb-3d.com/wordpress/wp-content/uploads/ipc-sm-782a_amendment_1_and_2.pdf), generated with kicad-footprint-generator")
 		(tags "capacitor")
@@
 	(footprint "Capacitor_SMD:C_0603_1608Metric"
 		(layer "F.Cu")
-		(at 180.6456 129.9422)
+		(at 222.1108 112.2638)
 		(descr "Capacitor SMD 0603 (1608 Metric), square (rectangular) end terminal, IPC-7351 nominal, (Body size source: IPC-SM-782 page 76, https://www.pcb-3d.com/wordpress/wp-content/uploads/ipc-sm-782a_amendment_1_and_2.pdf), generated with kicad-footprint-generator")
 		(tags "capacitor")
@@
 	(footprint "Resistor_SMD:R_0603_1608Metric"
 		(layer "F.Cu")
-		(at 174.2996 128.1336 180)
+		(at 215.7648 110.4552 180)
 		(descr "Resistor SMD 0603 (1608 Metric), square (rectangular) end terminal, IPC-7351 nominal, (Body size source: IPC-SM-782 page 72, https://www.pcb-3d.com/wordpress/wp-content/uploads/ipc-sm-782a_amendment_1_and_2.pdf), generated with kicad-footprint-generator")
 		(tags "resistor")
@@
 	(footprint "Resistor_SMD:R_0603_1608Metric"
 		(layer "F.Cu")
-		(at 190.5 116.3198 90)
+		(at 231.9652 98.6414 90)
 		(descr "Resistor SMD 0603 (1608 Metric), square (rectangular) end terminal, IPC-7351 nominal, (Body size source: IPC-SM-782 page 72, https://www.pcb-3d.com/wordpress/wp-content/uploads/ipc-sm-782a_amendment_1_and_2.pdf), generated with kicad-footprint-generator")
 		(tags "resistor")
@@
 	(footprint "Capacitor_SMD:C_0603_1608Metric"
 		(layer "F.Cu")
-		(at 189.9666 119.507 180)
+		(at 231.4318 101.8286 180)
 		(descr "Capacitor SMD 0603 (1608 Metric), square (rectangular) end terminal, IPC-7351 nominal, (Body size source: IPC-SM-782 page 76, https://www.pcb-3d.com/wordpress/wp-content/uploads/ipc-sm-782a_amendment_1_and_2.pdf), generated with kicad-footprint-generator")
 		(tags "capacitor")
@@
 	(footprint "Capacitor_SMD:C_0603_1608Metric"
 		(layer "F.Cu")
-		(at 188.1632 117.1204 180)
+		(at 229.6284 99.442 180)
 		(descr "Capacitor SMD 0603 (1608 Metric), square (rectangular) end terminal, IPC-7351 nominal, (Body size source: IPC-SM-782 page 76, https://www.pcb-3d.com/wordpress/wp-content/uploads/ipc-sm-782a_amendment_1_and_2.pdf), generated with kicad-footprint-generator")
 		(tags "capacitor")
