File: Board/KiCAD/Cell_Interface.kicad_sch (KiCad schematic)
At the start: 26 parts, among them Q23 2N7002, Q24 2N7002, Q25 2N7002, Q26 2N7002, Q5 BSS83P, Q6 BSS83P, Q7 BSS83P, Q8 BSS83P, U6 INA219AxDCN, U7 INA219AxDCN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

Commit message: revised PCB
This design accounts for majority of the updates requested by Faculty Advisor

@KeytarGoblin  @andrewgreenberg
Connections:
- net Cell 1: now also Q8.2 (S); no longer Q8.3 (D)
- net Cell 2: now also Q7.2 (S); no longer Q7.3 (D)
- net Cell 3: now also Q6.2 (S); no longer Q6.3 (D)
- net at R66.1: now also Q8.3 (D); no longer Q8.2 (S)
- net at R67.1: now also Q7.3 (D); no longer Q7.2 (S)
- net at R68.1: now also Q6.3 (D); no longer Q6.2 (S)
Changed lines of the file:
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@@
 		(lib_id "Transistor_FET:BSS83P")
 		(at 91.44 157.48 0)
-		(unit 1)
-		(exclude_from_sim no)
-		(in_bom yes)
-		(on_board yes)
-		(dnp no)
-		(fields_autoplaced yes)
+		(mirror x)
+		(unit 1)
+		(exclude_from_sim no)
+		(in_bom yes)
+		(on_board yes)
+		(dnp no)
 		(property "Reference" "Q8"
-			(at 97.79 156.2099 0)
+			(at 97.79 158.7501 0)
 			(effects
 				(font
@@
 		)
 		(property "Value" "BSS83P"
-			(at 97.79 158.7499 0)
+			(at 97.79 156.2101 0)
 			(effects
 				(font
@@
 		)
 		(property "Footprint" "Package_TO_SOT_SMD:SOT-23"
-			(at 96.52 159.385 0)
+			(at 96.52 155.575 0)
 			(effects
 				(font
@@
 		)
 		(property "Datasheet" "http://www.farnell.com/datasheets/1835997.pdf"
-			(at 96.52 161.29 0)
+			(at 96.52 153.67 0)
 			(effects
 				(font
@@
 		(lib_id "Transistor_FET:BSS83P")
 		(at 91.44 119.38 0)
-		(unit 1)
-		(exclude_from_sim no)
-		(in_bom yes)
-		(on_board yes)
-		(dnp no)
-		(fields_autoplaced yes)
+		(mirror x)
+		(unit 1)
+		(exclude_from_sim no)
+		(in_bom yes)
+		(on_board yes)
+		(dnp no)
 		(property "Reference" "Q7"
-			(at 97.79 118.1099 0)
+			(at 97.79 120.6501 0)
 			(effects
 				(font
@@
 		)
 		(property "Value" "BSS83P"
-			(at 97.79 120.6499 0)
+			(at 97.79 118.1101 0)
 			(effects
 				(font
@@
 		)
 		(property "Footprint" "Package_TO_SOT_SMD:SOT-23"
-			(at 96.52 121.285 0)
+			(at 96.52 117.475 0)
 			(effects
 				(font
@@
 		)
 		(property "Datasheet" "http://www.farnell.com/datasheets/1835997.pdf"
-			(at 96.52 123.19 0)
+			(at 96.52 115.57 0)
 			(effects
 				(font
@@
 		(lib_id "Transistor_FET:BSS83P")
 		(at 91.44 87.63 0)
-		(unit 1)
-		(exclude_from_sim no)
-		(in_bom yes)
-		(on_board yes)
-		(dnp no)
-		(fields_autoplaced yes)
+		(mirror x)
+		(unit 1)
+		(exclude_from_sim no)
+		(in_bom yes)
+		(on_board yes)
+		(dnp no)
 		(property "Reference" "Q6"
-			(at 97.79 86.3599 0)
+			(at 97.79 88.9001 0)
 			(effects
 				(font
@@
 		)
 		(property "Value" "BSS83P"
-			(at 97.79 88.8999 0)
+			(at 97.79 86.3601 0)
 			(effects
 				(font
@@
 		)
 		(property "Footprint" "Package_TO_SOT_SMD:SOT-23"
-			(at 96.52 89.535 0)
+			(at 96.52 85.725 0)
 			(effects
 				(font
@@
 		)
 		(property "Datasheet" "http://www.farnell.com/datasheets/1835997.pdf"
-			(at 96.52 91.44 0)
-			(effects
-				(font
+			(at 96.52 83.82 0)
+			(effects
+				(font
