File: Board/KiCAD/Battery_Management_System.kicad_sch (KiCad schematic)
At the start: 19 parts, among them J1 Conn_01x06_Socket, J10 Conn_01x02, J11 Conn_01x02, J12 Conn_01x02, J13 Conn_01x02, J5 Conn_01x03, J7 Conn_01x05, J8 Conn_01x02, J9 Conn_01x02

Commit message: Edits to PCB
@andrewgreenberg @KeytarGoblin
Connections:
- net Cell Interface/Cell 4 is gone; now on net Cell Interface/BATT: J7.1 (Pin_1)
Other:
- sheet Cell Interface ports: added none; removed Cell 4
Changed lines of the file:
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@@
+	)
+	(junction
+		(at 173.99 100.33)
+		(diameter 0)
+		(color 0 0 0 0)
 	)
 	(junction
@@
 	(wire
 		(pts
-			(xy 186.69 115.57) (xy 196.85 115.57)
-		)
-		(stroke
-			(width 0)
-			(type default)
-		)
-	)
-	(wire
-		(pts
 			(xy 77.47 85.09) (xy 69.85 85.09)
 		)
@@
 	(wire
 		(pts
+			(xy 189.23 115.57) (xy 189.23 100.33)
+		)
+		(stroke
+			(width 0)
+			(type default)
+		)
+	)
+	(wire
+		(pts
 			(xy 107.95 148.59) (xy 106.68 148.59)
 		)
@@
 	(wire
 		(pts
+			(xy 196.85 115.57) (xy 189.23 115.57)
+		)
+		(stroke
+			(width 0)
+			(type default)
+		)
+	)
+	(wire
+		(pts
 			(xy 62.23 114.3) (xy 62.23 113.03)
 		)
@@
 	(wire
 		(pts
-			(xy 173.99 88.9) (xy 173.99 102.87)
+			(xy 189.23 100.33) (xy 173.99 100.33)
+		)
+		(stroke
+			(width 0)
+			(type default)
+		)
+	)
+	(wire
+		(pts
+			(xy 173.99 88.9) (xy 173.99 100.33)
 		)
 		(stroke
@@
 		(pts
 			(xy 106.68 148.59) (xy 106.68 157.48)
+		)
+		(stroke
+			(width 0)
+			(type default)
+		)
+	)
+	(wire
+		(pts
+			(xy 173.99 100.33) (xy 173.99 102.87)
 		)
 		(stroke
@@
 			(effects
 				(font
-					(size 1.27 1.27)
-				)
-				(justify right)
-			)
-		)
-		(pin "Cell 4" input
-			(at 186.69 115.57 0)
-			(effects
-				(font

Commit message: Polish on schematic and board. Changed balance resistors to 100 ohms. Lots of silly OCD cleanup and documentation. Board has thicker (0.2mm) I2C lines, cleaned up 3.3V connections to reduce impedance, lots of other small tweaks.
Other:
- note added: "I2C to Host Microcontroller"
- note added: "Serial Debug (FT232RL 6pin)"
- note added: "To Host System Voltage: Vbatt or external power (switched) Current: **TBD** A max unless batteries have limit"
- note added: "To battey cells 1, 2, 3, or 4 cells (Na Ion, Li Ion, Other TBD!)"
- note removed: "Host Microcontroller"
- note removed: "Power out to Load"
- note removed: "SYSTEM OVERVIEW HERE PLZ"
- note removed: "To battey cells 1, 2, 3, or 4 cells"
- note removed: "USB to Serial Breaktout FT232RL"
- moved on the sheet: J1, J5, J9, TP24, TP25

Commit message: BOM Complete Need a Once Over Check
Parts:
- J1: MFR (none) -> Würth Elektronik; MPN (none) -> 732-5319-ND; Package (none) -> 61300611121
- J10, J11, J12, J13, J8, J9: MFR (none) -> TE Connectivity AMP Connectors; MPN (none) -> 5-146285-2-ND; Package (none) -> 5-146285-2
- J5: MFR (none) -> Würth Elektronik; MPN (none) -> 732-5316-ND; Package (none) -> 61300311121
- J7: MFR (none) -> Würth Elektronik; MPN (none) -> 732-5318-ND; Package (none) -> 61300511121
